Commit message: Added Hokuyo Laser Sensor

File: rotors_description/urdf/multirotor_base.xacro (robot description, xacro)
@@ -76,4 +76,67 @@
       </sensor>
     </gazebo>
+    <!-- attach hokuyo laser sensor -->
+      <joint name="hokuyo_joint" type="fixed">
+    <axis xyz="0 1 0" />
+    <origin xyz="0 0 0.08" rpy="0 0 0"/>
+    <parent link="${robot_namespace}/base_link"/>
+    <child link="hokuyo_link"/>
+  </joint>
+  <!-- Hokuyo Laser -->
+  <link name="hokuyo_link">
+    <collision>
+      <origin xyz="0 0 0" rpy="0 0 0"/>
+      <geometry>
+    <box size="0.1 0.1 0.1"/>
+      </geometry>
+    </collision>
+    <visual>
+      <origin xyz="0 0 0" rpy="0 0 0"/>
+      <geometry>
+        <mesh filename="package://rotors_description/meshes/hokuyo.dae"/>
+      </geometry>
+    </visual>
+    <inertial>
+      <mass value="1e-5" />
+      <origin xyz="0 0 0" rpy="0 0 0"/>
+      <inertia ixx="1e-6" ixy="0" ixz="0" iyy="1e-6" iyz="0" izz="1e-6" />
+    </inertial>
+  </link>
+    <!-- hokuyo plugin -->
+  <gazebo reference="hokuyo_link">
+    <sensor type="gpu_ray" name="head_hokuyo_sensor">
+      <pose>0 0 0 0 0 0</pose>
+      <visualize>true</visualize>
+      <update_rate>40</update_rate>
+      <ray>
+        <scan>
+          <horizontal>
+            <samples>20</samples>
+            <resolution>1</resolution>
+            <min_angle>-3.140796</min_angle>
+            <max_angle>3.140796</max_angle>
+          </horizontal>
+        </scan>
+        <range>
+          <min>0.10</min>
+          <max>3.0</max>
+          <resolution>0.01</resolution>
+        </range>
+        <noise>
+          <type>gaussian</type>
+          <!-- Noise parameters based on published spec for Hokuyo laser
+               achieving "+-30mm" accuracy at range < 10m.  A mean of 0.0m and
+               stddev of 0.01m will put 99.7% of samples within 0.03m of the true
+               reading. -->
+          <mean>0.0</mean>
+          <stddev>0.01</stddev>
+        </noise>
+      </ray>
+      <plugin name="gazebo_ros_head_hokuyo_controller" filename="libgazebo_ros_gpu_laser.so">
+        <topicName>/${robot_namespace}/laser/scan</topicName>
+        <frameName>hokuyo_link</frameName>
+      </plugin>
+    </sensor>
+  </gazebo>
     <!-- attach multirotor_base_plugin to the base_link -->
     <gazebo >

Commit message: added rpy values

File: rotors_description/urdf/multirotor_base.xacro (robot description, xacro)
@@ -43,5 +43,5 @@
       <inertial>
         <mass value="${mass}" />  <!-- [kg] -->
-        <origin xyz="0 0 0" />
+        <origin xyz="0 0 0" rpy="0 0 0" />
         <xacro:insert_block name="inertia" />
       </inertial>

File: rotors_gazebo/models/rotors_description/urdf/multirotor_base.xacro (robot description, xacro)
@@ -29,5 +29,5 @@
       <inertial>
         <mass value="${mass}" />  <!-- [kg] -->
-        <origin xyz="0 0 0" />
+        <origin xyz="0 0 0" rpy="0 0 0"/>
         <xacro:insert_block name="inertia" />
       </inertial>
