Commit message: added contact sensor with plugin, changed collision_box dimensions

File: rotors_description/urdf/bebop2.xacro (robot description, xacro)
@@ -8,4 +8,6 @@
   <xacro:property name="mass" value="0.503" /> <!-- [kg] -->
   <xacro:property name="body_width" value="0.316618" /> <!-- [m] -->
+  <xacro:property name="collision_width" value="0.36" /> <!-- [m] -->
+  <xacro:property name="collision_topic_name" value="/bebop2/base_link/collision_count" /> <!-- [m] -->
   <xacro:property name="body_height" value="0.089582" /> <!-- [m] -->
   <xacro:property name="mass_rotor" value="0.001" /> <!-- [kg] -->
@@ -38,4 +40,6 @@
     mass="${mass}"
     body_width="${body_width}"
+    collision_width="${collision_width}"
+    collision_topic_name="${collision_topic_name}"
     body_height="${body_height}"
     use_mesh_file="${use_mesh_file}"

File: rotors_description/urdf/multirotor_base.xacro (robot description, xacro)
@@ -33,5 +33,5 @@
   <!-- Main multirotor link -->
   <xacro:macro name="multirotor_base_macro"
-    params="robot_namespace mass body_width body_height use_mesh_file mesh_file *inertia">
+    params="robot_namespace mass body_width collision_width collision_topic_name body_height use_mesh_file mesh_file *inertia">
     <link name="${robot_namespace}/base_link"></link>
     <joint name="${robot_namespace}/base_joint" type="fixed">
@@ -57,13 +57,25 @@
         </geometry>
       </visual>
-      <collision>
+      <collision name="collision">
         <origin xyz="0 0 0" rpy="0 0 0" />
         <geometry>
-          <box size="${body_width} ${body_width} ${body_height}" /> <!-- [m] [m] [m] -->
+          <box size="${collision_width} ${collision_width} ${body_height}" /> <!-- [m] [m] [m] -->
         </geometry>
       </collision>
     </link>
+    <!-- collision sensor for the base link -->
+    <gazebo reference="${robot_namespace}/base_link_inertia">
+      <sensor name='contact' type='contact'>
+        <plugin name='contact' filename='libcontact.so'>
+          <TopicName>${collision_topic_name}</TopicName>
+        </plugin>
+        <contact>
+          <collision>${robot_namespace}/base_link_fixed_joint_lump__collision_collision</collision>
+          <topic>/robot/isworking</topic>
+        </contact>
+      </sensor>
+    </gazebo>
     <!-- attach multirotor_base_plugin to the base_link -->
-    <gazebo>
+    <gazebo >
       <plugin filename="librotors_gazebo_multirotor_base_plugin.so" name="multirotor_base_plugin">
         <robotNamespace>${robot_namespace}</robotNamespace>

Commit message: only_depth

File: rotors_description/urdf/bebop2.xacro (robot description, xacro)
@@ -8,5 +8,5 @@
   <xacro:property name="mass" value="0.503" /> <!-- [kg] -->
   <xacro:property name="body_width" value="0.316618" /> <!-- [m] -->
-  <xacro:property name="collision_width" value="0.36" /> <!-- [m] -->
+  <xacro:property name="collision_width" value="0.40" /> <!-- [m] -->
   <xacro:property name="collision_topic_name" value="/bebop2/base_link/collision_count" /> <!-- [m] -->
   <xacro:property name="body_height" value="0.089582" /> <!-- [m] -->

Commit message: distance env with 0 1 reward -100 collision reward fixed length

File: rotors_description/urdf/bebop2.xacro (robot description, xacro)
@@ -8,6 +8,6 @@
   <xacro:property name="mass" value="0.503" /> <!-- [kg] -->
   <xacro:property name="body_width" value="0.316618" /> <!-- [m] -->
+  <xacro:property name="collision_topic_name" value="/bebop2/base_link/collision_count" /> <!-- [m] -->
   <xacro:property name="collision_width" value="0.40" /> <!-- [m] -->
-  <xacro:property name="collision_topic_name" value="/bebop2/base_link/collision_count" /> <!-- [m] -->
   <xacro:property name="body_height" value="0.089582" /> <!-- [m] -->
   <xacro:property name="mass_rotor" value="0.001" /> <!-- [kg] -->

Commit message: distance_with_multi_with_gray_depth_latest_increased_sim15

File: rotors_description/urdf/bebop2.xacro (robot description, xacro)
@@ -3,5 +3,5 @@
   <!-- Properties -->
   <xacro:property name="namespace" value="$(arg namespace)" />
-  <xacro:property name="rotor_velocity_slowdown_sim" value="10" />
+  <xacro:property name="rotor_velocity_slowdown_sim" value="15" />
   <xacro:property name="use_mesh_file" value="true" />
   <xacro:property name="mesh_file" value="package://rotors_description/meshes/bebop2.dae" />
@@ -136,5 +136,5 @@
       parent_link="${namespace}/base_link"
       camera_suffix="base"
-      frame_rate="15"
+      frame_rate="20"
       horizontal_fov="1.7"
       image_height="50"
